File: ESP-WROOM-02-breakout.kicad_pcb (KiCad board)
At the start: 2 copper layers, 31.8 x 31.7 mm, 5 parts, among them P1 CONN_01X09, P2 CONN_01X09, U1 ESP-13-WROOM-02

Commit message: Add MCQN logo to the PCB silkscreen.
Parts:
- added G***: LOGO, MCQN Ltd:mcqn-logo-10mm, F.Cu at (134.6, 76.2)
Other:
- board text added: "r20160702"
- board text removed: "r20160601"
